Commit message: Improve Gazebo visuals and add project screenshot

File: src/mobile_robot_description/urdf/mobile_base.urdf.xacro (robot description, xacro)
@@ -352,3 +352,42 @@
   </plugin>
 </gazebo>
+  <!-- ================================= -->
+  <!-- Gazebo Visual Materials           -->
+  <!-- ================================= -->
+  <gazebo reference="base_link">
+    <material>Gazebo/DarkGrey</material>
+  </gazebo>
+  <gazebo reference="wheel_left_link">
+    <material>Gazebo/Black</material>
+  </gazebo>
+  <gazebo reference="wheel_right_link">
+    <material>Gazebo/Black</material>
+  </gazebo>
+  <gazebo reference="base_scan">
+    <material>Gazebo/DarkGrey</material>
+  </gazebo>
+  <!-- ================================= -->
+  <!-- Gazebo Visual Materials - Arm     -->
+  <!-- ================================= -->
+  <gazebo reference="link1">
+    <material>Gazebo/Grey</material>
+  </gazebo>
+  <gazebo reference="link2">
+    <material>Gazebo/Grey</material>
+  </gazebo>
+  <gazebo reference="link3">
+    <material>Gazebo/Grey</material>
+  </gazebo>
+  <gazebo reference="link4">
+    <material>Gazebo/DarkGrey</material>
+  </gazebo>
+  <gazebo reference="link5">
+    <material>Gazebo/DarkGrey</material>
+  </gazebo>
+  <gazebo reference="gripper_left_link">
+    <material>Gazebo/DarkGrey</material>
+  </gazebo>
+  <gazebo reference="gripper_right_link">
+    <material>Gazebo/DarkGrey</material>
+  </gazebo>
 </robot>

Commit message: Phase 3: integrate MoveIt 2 and stabilize Gazebo

File: src/mobile_robot_description/urdf/mobile_base.urdf.xacro (robot description, xacro)
@@ -154,9 +154,9 @@
   <link name="caster_back_right_link">
     <collision>
-      <origin xyz="0 0 0"/>
-      <geometry>
-        <sphere radius="0.010"/>
-      </geometry>
-   </collision>
+      <origin xyz="0 0.001 0" rpy="0 0 0"/>
+      <geometry>
+        <box size="0.030 0.009 0.020"/>
+      </geometry>
+    </collision>
     <inertial>
       <mass value="0.005"/>
@@ -178,7 +178,7 @@
   <link name="caster_back_left_link">
     <collision>
-      <origin xyz="0 0 0"/>
-      <geometry>
-        <sphere radius="0.010"/>
+      <origin xyz="0 0.001 0" rpy="0 0 0"/>
+      <geometry>
+        <box size="0.030 0.009 0.020"/>
       </geometry>
     </collision>
